Commit message: Control Attached Gripper Simultaneously

File: marsha_description/urdf/gripper.urdf.xacro (robot description, xacro)
@@ -1,5 +1,4 @@
 <?xml version="1.0" encoding="utf-8"?>
 <robot xmlns:xacro="http://www.ros.org/wiki/xacro" name="tundra_gripper">
-<link name="world"/>
 <link name="palm">
   <inertial>
@@ -25,9 +24,4 @@
   </collision>
 </link>
-<joint name="world_joint" type="fixed">
-  <parent link="world"/>
-  <child link="palm"/>
-  <origin xyz="0 0 0" rpy="0 0 0"/>
-</joint>
 <link name="actuator_1">
     <inertial>
