Commit message: Added arm2d2

File: arm2d2/arm2d2_description/urdf/arm1_gazebo.urdf.xacro (robot description, xacro)
@@ -1,8 +1,8 @@
 <?xml version="1.0" encoding="utf-8" ?>
 <!-- =================================================================================== -->
-<!-- |  This document was autogenerated by xacro from /home/satlab/catkin_ws/src/ar_mini_description/urdf/ar_mini.xacro | -->
+<!-- |  This document was autogenerated by xacro from /home/satlab/catkin_ws/src/arm2d2_description/urdf/arm2d2.xacro | -->
 <!-- |  EDITING THIS FILE BY HAND IS NOT RECOMMENDED                 | -->
 <!-- =================================================================================== -->
-<robot name="ar_mini">
+<robot name="arm2d2">
   <material name="silver">
     <color rgba="0.700 0.700 0.700 1.000" />
@@ -18,5 +18,5 @@
       <origin rpy="0 0 0" xyz="0 0 0" />
       <geometry>
-        <mesh filename="package://ar_mini_description/meshes/base_link.stl" scale="0.001 0.001 0.001" />
+        <mesh filename="package://arm2d2_description/meshes/base_link.stl" scale="0.001 0.001 0.001" />
       </geometry>
       <material name="silver" />
@@ -25,5 +25,5 @@
       <origin rpy="0 0 0" xyz="0 0 0" />
       <geometry>
-        <mesh filename="package://ar_mini_description/meshes/base_link.stl" scale="0.001 0.001 0.001" />
+        <mesh filename="package://arm2d2_description/meshes/base_link.stl" scale="0.001 0.001 0.001" />
       </geometry>
     </collision>
@@ -34,5 +34,5 @@
     <origin xyz="0 0 0" rpy="0 0 0"/>
   </joint>
-  <link name="link1">
+  <link name="link_1">
     <inertial>
       <origin rpy="0 0 0" xyz="-0.00789643305978462 0.002474313899377526 0.01425764348212194" />
@@ -43,5 +43,5 @@
       <origin rpy="0 0 0" xyz="0.003226 0.019004 -0.084836" />
       <geometry>
-        <mesh filename="package://ar_mini_description/meshes/link1_1.stl" scale="0.001 0.001 0.001" />
+        <mesh filename="package://arm2d2_description/meshes/link1_1.stl" scale="0.001 0.001 0.001" />
       </geometry>
       <material name="silver" />
@@ -50,16 +50,16 @@
       <origin rpy="0 0 0" xyz="0.003226 0.019004 -0.084836" />
       <geometry>
-        <mesh filename="package://ar_mini_description/meshes/link1_1.stl" scale="0.001 0.001 0.001" />
-      </geometry>
-    </collision>
-  </link>
-  <joint name="joint1" type="revolute">
+        <mesh filename="package://arm2d2_description/meshes/link1_1.stl" scale="0.001 0.001 0.001" />
+      </geometry>
+    </collision>
+  </link>
+  <joint name="joint_1" type="revolute">
     <origin rpy="0 0 0" xyz="-0.003226 -0.019004 0.084836" />
     <parent link="base_link" />
-    <child link="link1" />
+    <child link="link_1" />
     <axis xyz="-0.0 -0.0 1.0" />
     <limit effort="100" lower="-3.1415" upper="3.1415" velocity="100"/>
   </joint>
-  <link name="link2">
+  <link name="link_2">
     <inertial>
       <origin rpy="0 0 0" xyz="0.01898708853636933 -8.655304474807987e-06 0.04227958883013139" />
@@ -70,5 +70,5 @@
       <origin rpy="0 0 0" xyz="0.023226 0.006935 -0.127996" />
       <geometry>
-        <mesh filename="package://ar_mini_description/meshes/link2_1.stl" scale="0.001 0.001 0.001" />
+        <mesh filename="package://arm2d2_description/meshes/link2_1.stl" scale="0.001 0.001 0.001" />
       </geometry>
       <material name="silver" />
@@ -77,16 +77,16 @@
       <origin rpy="0 0 0" xyz="0.023226 0.006935 -0.127996" />
       <geometry>
-        <mesh filename="package://ar_mini_description/meshes/link2_1.stl" scale="0.001 0.001 0.001" />
-      </geometry>
-    </collision>
-  </link>
-  <joint name="joint2" type="revolute">
+        <mesh filename="package://arm2d2_description/meshes/link2_1.stl" scale="0.001 0.001 0.001" />
+      </geometry>
+    </collision>
+  </link>
+  <joint name="joint_2" type="revolute">
     <origin rpy="0 0 0" xyz="-0.02 0.012069 0.04316" />
-    <parent link="link1" />
-    <child link="link2" />
+    <parent link="link_1" />
+    <child link="link_2" />
     <axis xyz="1.0 -0.0 0.0" />
     <limit effort="100" lower="-1.658063" upper="1.658063" velocity="100" />
   </joint>
-  <link name="link3">
+  <link name="link_3">
     <inertial>
       <origin rpy="0 0 0" xyz="0.01486624761711016 5.106898781712457e-05 0.01728082961823646" />
@@ -97,5 +97,5 @@
       <origin rpy="0 0 0" xyz="0.013226 0.006935 -0.247996" />
       <geometry>
-        <mesh filename="package://ar_mini_description/meshes/link3_1.stl" scale="0.001 0.001 0.001" />
+        <mesh filename="package://arm2d2_description/meshes/link3_1.stl" scale="0.001 0.001 0.001" />
       </geometry>
       <material name="silver" />
@@ -104,9 +104,16 @@
       <origin rpy="0 0 0" xyz="0.013226 0.006935 -0.247996" />
       <geometry>
-        <mesh filename="package://ar_mini_description/meshes/link3_1.stl" scale="0.001 0.001 0.001" />
-      </geometry>
-    </collision>
-  </link>
-  <link name="link4">
+        <mesh filename="package://arm2d2_description/meshes/link3_1.stl" scale="0.001 0.001 0.001" />
+      </geometry>
+    </collision>
+  </link>
+  <joint name="joint_3" type="revolute">
+    <origin rpy="0 0 0" xyz="0.01 0.0 0.12" />
+    <parent link="link_2" />
+    <child link="link_3" />
+    <axis xyz="1.0 -0.0 0.0" />
+    <limit effort="100" lower="-2.268928" upper="2.268928" velocity="100" />
+  </joint>
+  <link name="link_4">
     <inertial>
       <origin rpy="0 0 0" xyz="-0.011101446329824061 3.2242915119862735e-05 0.04184113083783203" />
@@ -117,5 +124,5 @@
       <origin rpy="0 0 0" xyz="-0.006774 0.006935 -0.287996" />
       <geometry>
-        <mesh filename="package://ar_mini_description/meshes/link4_1.stl" scale="0.001 0.001 0.001" />
+        <mesh filename="package://arm2d2_description/meshes/link4_1.stl" scale="0.001 0.001 0.001" />
       </geometry>
       <material name="silver" />
@@ -124,8 +131,15 @@
       <origin rpy="0 0 0" xyz="-0.006774 0.006935 -0.287996" />
       <geometry>
-        <mesh filename="package://ar_mini_description/meshes/link4_1.stl" scale="0.001 0.001 0.001" />
-      </geometry>
-    </collision>
-  </link>
+        <mesh filename="package://arm2d2_description/meshes/link4_1.stl" scale="0.001 0.001 0.001" />
+      </geometry>
+    </collision>
+  </link>
+  <joint name="joint_4" type="revolute">
+    <origin rpy="0 0 0" xyz="0.02 0.0 0.04" />
+    <parent link="link_3" />
+    <child link="link_4" />
+    <axis xyz="0.0 7e-06 1.0" />
+    <limit effort="100" lower="-3.1415" upper="3.1415" velocity="100"/>
+  </joint>
   <link name="palm">
     <inertial>
@@ -137,5 +151,5 @@
       <origin rpy="0 0 0" xyz="0.003226 0.006934 -0.377996" />
       <geometry>
-        <mesh filename="package://ar_mini_description/meshes/palm_1.stl" scale="0.001 0.001 0.001" />
+        <mesh filename="package://arm2d2_description/meshes/palm_1.stl" scale="0.001 0.001 0.001" />
       </geometry>
       <material name="silver" />
@@ -144,8 +158,16 @@
       <origin rpy="0 0 0" xyz="0.003226 0.006934 -0.377996" />
       <geometry>
-        <mesh filename="package://ar_mini_description/meshes/palm_1.stl" scale="0.001 0.001 0.001" />
-      </geometry>
-    </collision>
-  </link>
+        <mesh filename="package://arm2d2_description/meshes/palm_1.stl" scale="0.001 0.001 0.001" />
+      </geometry>
+    </collision>
+  </link>
+  <joint name="joint_5" type="revolute">
+    <origin rpy="0 0 0" xyz="-0.01 1e-06 0.09" />
+    <parent link="link_4" />
+    <child link="palm" />
+    <axis xyz="1.0 -0.0 0.0" />
+    <limit effort="100" lower="-2.268928" upper="2.268928" velocity="100" />
+  </joint>
+  <!--
   <link name="finger_1">
     <inertial>
@@ -157,5 +179,5 @@
       <origin rpy="0 0 0" xyz="-0.038503 0.023636 -0.424996" />
       <geometry>
-        <mesh filename="package://ar_mini_description/meshes/finger_1.stl" scale="0.001 0.001 0.001" />
+        <mesh filename="package://arm2d2_description/meshes/finger_1.stl" scale="0.001 0.001 0.001" />
       </geometry>
       <material name="silver" />
@@ -164,69 +186,8 @@
       <origin rpy="0 0 0" xyz="-0.038503 0.023636 -0.424996" />
       <geometry>
-        <mesh filename="package://ar_mini_description/meshes/finger_1.stl" scale="0.001 0.001 0.001" />
-      </geometry>
-    </collision>
-  </link>
-  <link name="finger_2">
-    <inertial>
-      <origin rpy="0 0 0" xyz="-0.0021646025973648094 0.00567892122346535 0.027279474187493602" />
-      <mass value="0.005277222771828628" />
-      <inertia ixx="2e-06" ixy="-0.0" ixz="-0.0" iyy="2e-06" iyz="-0.0" izz="0.0" />
-    </inertial>
-    <visual>
-      <origin rpy="0 0 0" xyz="-0.005046 0.023636 -0.424996" />
-      <geometry>
-        <mesh filename="package://ar_mini_description/meshes/finger_2.stl" scale="0.001 0.001 0.001" />
-      </geometry>
-      <material name="silver" />
-    </visual>
-    <collision>
-      <origin rpy="0 0 0" xyz="-0.005046 0.023636 -0.424996" />
-      <geometry>
-        <mesh filename="package://ar_mini_description/meshes/finger_2.stl" scale="0.001 0.001 0.001" />
-      </geometry>
-    </collision>
-  </link>
-  <link name="finger_3">
-    <inertial>
-      <origin rpy="0 0 0" xyz="0.006000455462889673 -0.000964137225942182 0.02727923439293578" />
-      <mass value="0.005277222771828628" />
-      <inertia ixx="2e-06" ixy="0.0" ixz="0.0" iyy="2e-06" iyz="0.0" izz="0.0" />
-    </inertial>
-    <visual>
-      <origin rpy="0 0 0" xyz="-0.015674 -0.015904 -0.424996" />
-      <geometry>
-        <mesh filename="package://ar_mini_description/meshes/finger_3.stl" scale="0.001 0.001 0.001" />
-      </geometry>
-      <material name="silver" />
-    </visual>
-    <collision>
-      <origin rpy="0 0 0" xyz="-0.015674 -0.015904 -0.424996" />
-      <geometry>
-        <mesh filename="package://ar_mini_description/meshes/finger_3.stl" scale="0.001 0.001 0.001" />
-      </geometry>
-    </collision>
-  </link>
-  <joint name="joint3" type="revolute">
-    <origin rpy="0 0 0" xyz="0.01 0.0 0.12" />
-    <parent link="link2" />
-    <child link="link3" />
-    <axis xyz="1.0 -0.0 0.0" />
-    <limit effort="100" lower="-2.268928" upper="2.268928" velocity="100" />
-  </joint>
-  <joint name="joint4" type="revolute">
-    <origin rpy="0 0 0" xyz="0.02 0.0 0.04" />
-    <parent link="link3" />
-    <child link="link4" />
-    <axis xyz="0.0 7e-06 1.0" />
-    <limit effort="100" lower="-3.1415" upper="3.1415" velocity="100"/>
-  </joint>
-  <joint name="joint5" type="revolute">
-    <origin rpy="0 0 0" xyz="-0.01 1e-06 0.09" />
-    <parent link="link4" />
-    <child link="palm" />
-    <axis xyz="1.0 -0.0 0.0" />
-    <limit effort="100" lower="-2.268928" upper="2.268928" velocity="100" />
-  </joint>
+        <mesh filename="package://arm2d2_description/meshes/finger_1.stl" scale="0.001 0.001 0.001" />
+      </geometry>
+    </collision>
+  </link>
   <joint name="finger_joint1" type="revolute">
     <origin rpy="0 0 0" xyz="0.041729 -0.016702 0.047" />
@@ -236,4 +197,24 @@
     <limit effort="100" lower="-0.698132" upper="0.0" velocity="100" />
   </joint>
+  <link name="finger_2">
+    <inertial>
+      <origin rpy="0 0 0" xyz="-0.0021646025973648094 0.00567892122346535 0.027279474187493602" />
+      <mass value="0.005277222771828628" />
+      <inertia ixx="2e-06" ixy="-0.0" ixz="-0.0" iyy="2e-06" iyz="-0.0" izz="0.0" />
+    </inertial>
+    <visual>
+      <origin rpy="0 0 0" xyz="-0.005046 0.023636 -0.424996" />
+      <geometry>
+        <mesh filename="package://arm2d2_description/meshes/finger_2.stl" scale="0.001 0.001 0.001" />
+      </geometry>
+      <material name="silver" />
+    </visual>
+    <collision>
+      <origin rpy="0 0 0" xyz="-0.005046 0.023636 -0.424996" />
+      <geometry>
+        <mesh filename="package://arm2d2_description/meshes/finger_2.stl" scale="0.001 0.001 0.001" />
+      </geometry>
+    </collision>
+  </link>
   <joint name="finger_joint2" type="revolute">
     <origin rpy="0 0 0" xyz="0.008272 -0.016702 0.047" />
@@ -243,4 +224,24 @@
     <limit effort="100" lower="0.0" upper="0.698132" velocity="100" />
   </joint>
+  <link name="finger_3">
+    <inertial>
+      <origin rpy="0 0 0" xyz="0.006000455462889673 -0.000964137225942182 0.02727923439293578" />
+      <mass value="0.005277222771828628" />
+      <inertia ixx="2e-06" ixy="0.0" ixz="0.0" iyy="2e-06" iyz="0.0" izz="0.0" />
+    </inertial>
+    <visual>
+      <origin rpy="0 0 0" xyz="-0.015674 -0.015904 -0.424996" />
+      <geometry>
+        <mesh filename="package://arm2d2_description/meshes/finger_3.stl" scale="0.001 0.001 0.001" />
+      </geometry>
+      <material name="silver" />
+    </visual>
+    <collision>
+      <origin rpy="0 0 0" xyz="-0.015674 -0.015904 -0.424996" />
+      <geometry>
+        <mesh filename="package://arm2d2_description/meshes/finger_3.stl" scale="0.001 0.001 0.001" />
+      </geometry>
+    </collision>
+  </link>
   <joint name="finger_joint3" type="revolute">
     <origin rpy="0 0 0" xyz="0.0189 0.022838 0.047" />
@@ -250,51 +251,63 @@
     <limit effort="100" lower="0.0" upper="0.698132" velocity="100" />
   </joint>
-  <transmission name="trans_joint2">
-    <type>transmission_interface/SimpleTransmission</type>
-    <joint name="joint2">
-      <hardwareInterface>hardware_interface/EffortJointInterface</hardwareInterface>
-    </joint>
-    <actuator name="joint2_motor">
-      <hardwareInterface>hardware_interface/EffortJointInterface</hardwareInterface>
-      <mechanicalReduction>1</mechanicalReduction>
-    </actuator>
-  </transmission>
-  <transmission name="trans_joint3">
-    <type>transmission_interface/SimpleTransmission</type>
-    <joint name="joint3">
-      <hardwareInterface>hardware_interface/EffortJointInterface</hardwareInterface>
-    </joint>
-    <actuator name="joint3_motor">
-      <hardwareInterface>hardware_interface/EffortJointInterface</hardwareInterface>
-      <mechanicalReduction>1</mechanicalReduction>
-    </actuator>
-  </transmission>
-  <transmission name="trans_joint4">
-    <type>transmission_interface/SimpleTransmission</type>
-    <joint name="joint4">
-      <hardwareInterface>hardware_interface/EffortJointInterface</hardwareInterface>
-    </joint>
-    <actuator name="joint4_motor">
-      <hardwareInterface>hardware_interface/EffortJointInterface</hardwareInterface>
-      <mechanicalReduction>1</mechanicalReduction>
-    </actuator>
-  </transmission>
-  <transmission name="trans_joint5">
-    <type>transmission_interface/SimpleTransmission</type>
-    <joint name="joint5">
-      <hardwareInterface>hardware_interface/EffortJointInterface</hardwareInterface>
-    </joint>
-    <actuator name="joint5_motor">
-      <hardwareInterface>hardware_interface/EffortJointInterface</hardwareInterface>
-      <mechanicalReduction>1</mechanicalReduction>
-    </actuator>
-  </transmission>
+  -->
+  <transmission name="transmission_1">
+    <type>transmission_interface/SimpleTransmission</type>
+    <joint name="joint_1">
+      <hardwareInterface>hardware_interface/PositionJointInterface</hardwareInterface>
+    </joint>
+    <actuator name="motor_1">
+      <hardwareInterface>hardware_interface/PositionJointInterface</hardwareInterface>
+      <mechanicalReduction>1</mechanicalReduction>
+    </actuator>
+  </transmission>
+  <transmission name="transmission_2">
+    <type>transmission_interface/SimpleTransmission</type>
+    <joint name="joint_2">
+      <hardwareInterface>hardware_interface/PositionJointInterface</hardwareInterface>
+    </joint>
+    <actuator name="motor_2">
+      <hardwareInterface>hardware_interface/PositionJointInterface</hardwareInterface>
+      <mechanicalReduction>1</mechanicalReduction>
+    </actuator>
+  </transmission>
+  <transmission name="transmission_3">
+    <type>transmission_interface/SimpleTransmission</type>
+    <joint name="joint_3">
+      <hardwareInterface>hardware_interface/PositionJointInterface</hardwareInterface>
+    </joint>
+    <actuator name="motor_3">
+      <hardwareInterface>hardware_interface/PositionJointInterface</hardwareInterface>
+      <mechanicalReduction>1</mechanicalReduction>
+    </actuator>
+  </transmission>
+  <transmission name="transmission_4">
+    <type>transmission_interface/SimpleTransmission</type>
+    <joint name="joint_4">
+      <hardwareInterface>hardware_interface/PositionJointInterface</hardwareInterface>
+    </joint>
+    <actuator name="motor_4">
+      <hardwareInterface>hardware_interface/PositionJointInterface</hardwareInterface>
+      <mechanicalReduction>1</mechanicalReduction>
+    </actuator>
+  </transmission>
+  <transmission name="transmission_5">
+    <type>transmission_interface/SimpleTransmission</type>
+    <joint name="joint_5">
+      <hardwareInterface>hardware_interface/PositionJointInterface</hardwareInterface>
+    </joint>
+    <actuator name="motor_5">
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