Commit message: Added arm2d2

File: arm2d2/arm2d2_description/urdf/arm2d2.urdf.xacro (robot description, xacro)
@@ -1,7 +1,7 @@
 <?xml version="1.0" ?>
-<robot name="ar_mini" xmlns:xacro="http://www.ros.org/wiki/xacro">
-<xacro:include filename="$(find ar_mini_description)/urdf/materials.xacro" />
-<xacro:include filename="$(find ar_mini_description)/urdf/ar_mini.trans" />
-<xacro:include filename="$(find ar_mini_description)/urdf/ar_mini.gazebo" />
+<robot name="arm2d2" xmlns:xacro="http://www.ros.org/wiki/xacro">
+<xacro:include filename="$(find arm2d2_description)/urdf/materials.xacro" />
+<xacro:include filename="$(find arm2d2_description)/urdf/arm2d2.trans" />
+<xacro:include filename="$(find arm2d2_description)/urdf/arm2d2.gazebo" />
 <link name="world"/>
 <link name="base_link">
@@ -14,5 +14,5 @@
     <origin rpy="0 0 0" xyz="0 0 0"/>
     <geometry>
-      <mesh filename="package://ar_mini_description/meshes/base_link.stl" scale="0.001 0.001 0.001"/>
+      <mesh filename="package://arm2d2_description/meshes/base_link.stl" scale="0.001 0.001 0.001"/>
     </geometry>
     <material name="silver"/>
@@ -21,5 +21,5 @@
     <origin rpy="0 0 0" xyz="0 0 0"/>
     <geometry>
-      <mesh filename="package://ar_mini_description/meshes/base_link.stl" scale="0.001 0.001 0.001"/>
+      <mesh filename="package://arm2d2_description/meshes/base_link.stl" scale="0.001 0.001 0.001"/>
     </geometry>
   </collision>
@@ -39,5 +39,5 @@
     <origin rpy="0 0 0" xyz="0.023226 0.006935 -0.127996"/>
     <geometry>
-      <mesh filename="package://ar_mini_description/meshes/link2_1.stl" scale="0.001 0.001 0.001"/>
+      <mesh filename="package://arm2d2_description/meshes/link2_1.stl" scale="0.001 0.001 0.001"/>
     </geometry>
     <material name="silver"/>
@@ -46,5 +46,5 @@
     <origin rpy="0 0 0" xyz="0.023226 0.006935 -0.127996"/>
     <geometry>
-      <mesh filename="package://ar_mini_description/meshes/link2_1.stl" scale="0.001 0.001 0.001"/>
+      <mesh filename="package://arm2d2_description/meshes/link2_1.stl" scale="0.001 0.001 0.001"/>
     </geometry>
   </collision>
@@ -59,5 +59,5 @@
     <origin rpy="0 0 0" xyz="0.013226 0.006935 -0.247996"/>
     <geometry>
-      <mesh filename="package://ar_mini_description/meshes/link3_1.stl" scale="0.001 0.001 0.001"/>
+      <mesh filename="package://arm2d2_description/meshes/link3_1.stl" scale="0.001 0.001 0.001"/>
     </geometry>
     <material name="silver"/>
@@ -66,5 +66,5 @@
     <origin rpy="0 0 0" xyz="0.013226 0.006935 -0.247996"/>
     <geometry>
-      <mesh filename="package://ar_mini_description/meshes/link3_1.stl" scale="0.001 0.001 0.001"/>
+      <mesh filename="package://arm2d2_description/meshes/link3_1.stl" scale="0.001 0.001 0.001"/>
     </geometry>
   </collision>
@@ -79,5 +79,5 @@
     <origin rpy="0 0 0" xyz="-0.006774 0.006935 -0.287996"/>
     <geometry>
-      <mesh filename="package://ar_mini_description/meshes/link4_1.stl" scale="0.001 0.001 0.001"/>
+      <mesh filename="package://arm2d2_description/meshes/link4_1.stl" scale="0.001 0.001 0.001"/>
     </geometry>
     <material name="silver"/>
@@ -86,5 +86,5 @@
     <origin rpy="0 0 0" xyz="-0.006774 0.006935 -0.287996"/>
     <geometry>
-      <mesh filename="package://ar_mini_description/meshes/link4_1.stl" scale="0.001 0.001 0.001"/>
+      <mesh filename="package://arm2d2_description/meshes/link4_1.stl" scale="0.001 0.001 0.001"/>
     </geometry>
   </collision>
@@ -99,5 +99,5 @@
     <origin rpy="0 0 0" xyz="0.003226 0.006934 -0.377996"/>
     <geometry>
-      <mesh filename="package://ar_mini_description/meshes/palm_1.stl" scale="0.001 0.001 0.001"/>
+      <mesh filename="package://arm2d2_description/meshes/palm_1.stl" scale="0.001 0.001 0.001"/>
     </geometry>
     <material name="silver"/>
@@ -106,5 +106,5 @@
     <origin rpy="0 0 0" xyz="0.003226 0.006934 -0.377996"/>
     <geometry>
-      <mesh filename="package://ar_mini_description/meshes/palm_1.stl" scale="0.001 0.001 0.001"/>
+      <mesh filename="package://arm2d2_description/meshes/palm_1.stl" scale="0.001 0.001 0.001"/>
     </geometry>
   </collision>
@@ -119,5 +119,5 @@
     <origin rpy="0 0 0" xyz="-0.038503 0.023636 -0.424996"/>
     <geometry>
-      <mesh filename="package://ar_mini_description/meshes/finger_1.stl" scale="0.001 0.001 0.001"/>
+      <mesh filename="package://arm2d2_description/meshes/finger_1.stl" scale="0.001 0.001 0.001"/>
     </geometry>
     <material name="silver"/>
@@ -126,5 +126,5 @@
     <origin rpy="0 0 0" xyz="-0.038503 0.023636 -0.424996"/>
     <geometry>
-      <mesh filename="package://ar_mini_description/meshes/finger_1.stl" scale="0.001 0.001 0.001"/>
+      <mesh filename="package://arm2d2_description/meshes/finger_1.stl" scale="0.001 0.001 0.001"/>
     </geometry>
   </collision>
@@ -139,5 +139,5 @@
     <origin rpy="0 0 0" xyz="-0.005046 0.023636 -0.424996"/>
     <geometry>
-      <mesh filename="package://ar_mini_description/meshes/finger_2.stl" scale="0.001 0.001 0.001"/>
+      <mesh filename="package://arm2d2_description/meshes/finger_2.stl" scale="0.001 0.001 0.001"/>
     </geometry>
     <material name="silver"/>
@@ -146,5 +146,5 @@
     <origin rpy="0 0 0" xyz="-0.005046 0.023636 -0.424996"/>
     <geometry>
-      <mesh filename="package://ar_mini_description/meshes/finger_2.stl" scale="0.001 0.001 0.001"/>
+      <mesh filename="package://arm2d2_description/meshes/finger_2.stl" scale="0.001 0.001 0.001"/>
     </geometry>
   </collision>
@@ -159,5 +159,5 @@
     <origin rpy="0 0 0" xyz="-0.015674 -0.015904 -0.424996"/>
     <geometry>
-      <mesh filename="package://ar_mini_description/meshes/finger_3.stl" scale="0.001 0.001 0.001"/>
+      <mesh filename="package://arm2d2_description/meshes/finger_3.stl" scale="0.001 0.001 0.001"/>
     </geometry>
     <material name="silver"/>
@@ -166,5 +166,5 @@
     <origin rpy="0 0 0" xyz="-0.015674 -0.015904 -0.424996"/>
     <geometry>
-      <mesh filename="package://ar_mini_description/meshes/finger_3.stl" scale="0.001 0.001 0.001"/>
+      <mesh filename="package://arm2d2_description/meshes/finger_3.stl" scale="0.001 0.001 0.001"/>
     </geometry>
   </collision>
@@ -179,5 +179,5 @@
     <origin rpy="0 0 0" xyz="0.003226 0.019004 -0.084836"/>
     <geometry>
-      <mesh filename="package://ar_mini_description/meshes/link1_1.stl" scale="0.001 0.001 0.001"/>
+      <mesh filename="package://arm2d2_description/meshes/link1_1.stl" scale="0.001 0.001 0.001"/>
     </geometry>
     <material name="silver"/>
@@ -186,5 +186,5 @@
     <origin rpy="0 0 0" xyz="0.003226 0.019004 -0.084836"/>
     <geometry>
-      <mesh filename="package://ar_mini_description/meshes/link1_1.stl" scale="0.001 0.001 0.001"/>
+      <mesh filename="package://arm2d2_description/meshes/link1_1.stl" scale="0.001 0.001 0.001"/>
     </geometry>
   </collision>

File: arm2d2/arm2d2_description/urdf/materials.xacro (robot description, xacro)
@@ -1,4 +1,4 @@
 <?xml version="1.0" ?>
-<robot name="ar_mini" xmlns:xacro="http://www.ros.org/wiki/xacro" >
+<robot name="arm2d2" xmlns:xacro="http://www.ros.org/wiki/xacro" >
 <material name="silver">
   <color rgba="0.700 0.700 0.700 1.000"/>

File: arm2d2/arm2d2_description/urdf/tundra_gazebo.urdf.xacro (robot description, xacro)
@@ -18,5 +18,5 @@
       <origin rpy="0 0 0" xyz="0.003226 0.006934 -0.377996"/>
       <geometry>
-        <mesh filename="package://ar_mini_description/meshes/palm_1.stl" scale="0.001 0.001 0.001"/>
+        <mesh filename="package://arm2d2_description/meshes/palm_1.stl" scale="0.001 0.001 0.001"/>
       </geometry>
       <material name="silver"/>
@@ -25,5 +25,5 @@
       <origin rpy="0 0 0" xyz="0.003226 0.006934 -0.377996"/>
       <geometry>
-        <mesh filename="package://ar_mini_description/meshes/palm_1.stl" scale="0.001 0.001 0.001"/>
+        <mesh filename="package://arm2d2_description/meshes/palm_1.stl" scale="0.001 0.001 0.001"/>
       </geometry>
     </collision>
@@ -43,5 +43,5 @@
       <origin rpy="0 0 0" xyz="-0.038503 0.023636 -0.424996"/>
       <geometry>
-        <mesh filename="package://ar_mini_description/meshes/finger_1.stl" scale="0.001 0.001 0.001"/>
+        <mesh filename="package://arm2d2_description/meshes/finger_1.stl" scale="0.001 0.001 0.001"/>
       </geometry>
       <material name="silver"/>
@@ -50,5 +50,5 @@
       <origin rpy="0 0 0" xyz="-0.038503 0.023636 -0.424996"/>
       <geometry>
-        <mesh filename="package://ar_mini_description/meshes/finger_1.stl" scale="0.001 0.001 0.001"/>
+        <mesh filename="package://arm2d2_description/meshes/finger_1.stl" scale="0.001 0.001 0.001"/>
       </geometry>
     </collision>
@@ -70,5 +70,5 @@
       <origin rpy="0 0 0" xyz="-0.005046 0.023636 -0.424996"/>
       <geometry>
-        <mesh filename="package://ar_mini_description/meshes/finger_2.stl" scale="0.001 0.001 0.001"/>
+        <mesh filename="package://arm2d2_description/meshes/finger_2.stl" scale="0.001 0.001 0.001"/>
       </geometry>
       <material name="silver"/>
@@ -77,5 +77,5 @@
       <origin rpy="0 0 0" xyz="-0.005046 0.023636 -0.424996"/>
       <geometry>
-        <mesh filename="package://ar_mini_description/meshes/finger_2.stl" scale="0.001 0.001 0.001"/>
+        <mesh filename="package://arm2d2_description/meshes/finger_2.stl" scale="0.001 0.001 0.001"/>
       </geometry>
     </collision>
@@ -97,5 +97,5 @@
       <origin rpy="0 0 0" xyz="-0.015674 -0.015904 -0.424996"/>
       <geometry>
-        <mesh filename="package://ar_mini_description/meshes/finger_3.stl" scale="0.001 0.001 0.001"/>
+        <mesh filename="package://arm2d2_description/meshes/finger_3.stl" scale="0.001 0.001 0.001"/>
       </geometry>
       <material name="silver"/>
@@ -104,5 +104,5 @@
       <origin rpy="0 0 0" xyz="-0.015674 -0.015904 -0.424996"/>
       <geometry>
-        <mesh filename="package://ar_mini_description/meshes/finger_3.stl" scale="0.001 0.001 0.001"/>
+        <mesh filename="package://arm2d2_description/meshes/finger_3.stl" scale="0.001 0.001 0.001"/>
       </geometry>
     </collision>

Commit message: AR3 arm & gripper work, ARM2D2 single arm & gripper work

File: arm2d2/arm2d2_description/urdf/arm1_gazebo.urdf.xacro (robot description, xacro)
@@ -142,5 +142,5 @@
     <limit effort="100" lower="-3.1415" upper="3.1415" velocity="100"/>
   </joint>
-  <link name="palm">
+  <link name="link_5">
     <inertial>
       <origin rpy="0 0 0" xyz="0.02043962300807103 -1.5866844334157942e-07 0.010610125536728798" />
@@ -151,5 +151,5 @@
       <origin rpy="0 0 0" xyz="0.003226 0.006934 -0.377996" />
       <geometry>
-        <mesh filename="package://arm2d2_description/meshes/palm_1.stl" scale="0.001 0.001 0.001" />
+        <mesh filename="package://arm2d2_description/meshes/link_5.stl" scale="0.001 0.001 0.001" />
       </geometry>
       <material name="silver" />
@@ -158,5 +158,5 @@
       <origin rpy="0 0 0" xyz="0.003226 0.006934 -0.377996" />
       <geometry>
-        <mesh filename="package://arm2d2_description/meshes/palm_1.stl" scale="0.001 0.001 0.001" />
+        <mesh filename="package://arm2d2_description/meshes/link_5.stl" scale="0.001 0.001 0.001" />
       </geometry>
     </collision>
@@ -165,5 +165,5 @@
     <origin rpy="0 0 0" xyz="-0.01 1e-06 0.09" />
     <parent link="link_4" />
-    <child link="palm" />
+    <child link="link_5" />
     <axis xyz="1.0 -0.0 0.0" />
     <limit effort="100" lower="-2.268928" upper="2.268928" velocity="100" />

File: arm2d2/arm2d2_description/urdf/arm2d2.xacro (robot description, xacro)
@@ -15,5 +15,5 @@
   <!-- Include arm and gripper urdfs-->
   <xacro:if value="$(arg include_arm)">
-    <xacro:include filename="$(find arm2d2_description)/urdf/arm1.urdf.xacro"/>
+    <xacro:include filename="$(find arm2d2_description)/urdf/arm1_gazebo.urdf.xacro"/>
   </xacro:if>
   <xacro:if value="$(arg include_gripper)">
@@ -25,5 +25,5 @@
       <joint name="gripper_joint" type="fixed">
         <parent link="link_5"/>
-        <child link="palm"/>
+        <child link="gripper_link"/>
         <xacro:if value="${is_left}">
           <origin xyz="0.025 0 0.025" rpy="0 0 0"/>
