Commit message: Both arm2d2s controlled manually simultaneously w/ grippers

File: arm2d2/arm2d2_description/urdf/arm1_gazebo.urdf.xacro (robot description, xacro)
@@ -1,64 +1,100 @@
 <?xml version="1.0" encoding="utf-8" ?>
-<!-- =================================================================================== -->
-<!-- |  This document was autogenerated by xacro from /home/satlab/catkin_ws/src/arm2d2_description/urdf/arm2d2.xacro | -->
-<!-- |  EDITING THIS FILE BY HAND IS NOT RECOMMENDED                 | -->
-<!-- =================================================================================== -->
-<robot name="arm2d2">
+<robot name="arm2d2" xmlns:xacro="http://www.ros.org/wifi/xacro">
+  <xacro:arg name="include_arm_base" default="true"/>
+  <xacro:arg name="ns" default="left"/>
+  <!-- Convert arg to property -->
+  <xacro:property name="ns" value="$(arg ns)"/>
   <material name="silver">
     <color rgba="0.700 0.700 0.700 1.000" />
   </material>
-  <link name="world"/>
-  <link name="base_link">
-    <inertial>
-      <origin rpy="0 0 0" xyz="0.06696356678870652 -0.08502272940883449 0.07176385561356924" />
-      <mass value="4.417422130393931" />
-      <inertia ixx="0.059227" ixy="0.000472" ixz="-0.000223" iyy="0.061578" iyz="0.000762" izz="0.075336" />
-    </inertial>
-    <visual>
-      <origin rpy="0 0 0" xyz="0 0 0" />
-      <geometry>
-        <mesh filename="package://arm2d2_description/meshes/base_link.stl" scale="0.001 0.001 0.001" />
-      </geometry>
-      <material name="silver" />
-    </visual>
-    <collision>
-      <origin rpy="0 0 0" xyz="0 0 0" />
-      <geometry>
-        <mesh filename="package://arm2d2_description/meshes/base_link.stl" scale="0.001 0.001 0.001" />
-      </geometry>
-    </collision>
-  </link>
-  <joint name="world_joint" type="fixed">
-    <parent link="world"/>
-    <child link="base_link"/>
-    <origin xyz="0 0 0" rpy="0 0 0"/>
-  </joint>
-  <link name="link_1">
-    <inertial>
-      <origin rpy="0 0 0" xyz="-0.00789643305978462 0.002474313899377526 0.01425764348212194" />
-      <mass value="0.17435766910618158" />
-      <inertia ixx="9.7e-05" ixy="7e-06" ixz="2.8e-05" iyy="0.000111" iyz="-1.2e-05" izz="0.000119" />
-    </inertial>
-    <visual>
-      <origin rpy="0 0 0" xyz="0.003226 0.019004 -0.084836" />
-      <geometry>
-        <mesh filename="package://arm2d2_description/meshes/link1_1.stl" scale="0.001 0.001 0.001" />
-      </geometry>
-      <material name="silver" />
-    </visual>
-    <collision>
-      <origin rpy="0 0 0" xyz="0.003226 0.019004 -0.084836" />
-      <geometry>
-        <mesh filename="package://arm2d2_description/meshes/link1_1.stl" scale="0.001 0.001 0.001" />
-      </geometry>
-    </collision>
-  </link>
-  <joint name="joint_1" type="revolute">
-    <origin rpy="0 0 0" xyz="-0.003226 -0.019004 0.084836" />
-    <parent link="base_link" />
-    <child link="link_1" />
-    <axis xyz="-0.0 -0.0 1.0" />
-    <limit effort="100" lower="-3.1415" upper="3.1415" velocity="100"/>
-  </joint>
+  <xacro:if value="$(arg include_arm_base)">
+    <xacro:include filename="$(find arm2d2_description)/urdf/base.urdf.xacro"/>
+  </xacro:if>
+  <xacro:unless value="$(arg include_arm_base)">
+    <link name="world"/>
+    <link name="base_link">
+      <inertial>
+        <origin rpy="0 0 0" xyz="0.06861790086338357 -0.0835697992386399 0.07107579694115096"/>
+        <mass value="4.519107238213137"/>
+        <inertia ixx="0.059779" ixy="-0.0" ixz="0.0" iyy="0.062251" iyz="0.000956" izz="0.076317"/>
+      </inertial>
+      <visual>
+        <origin rpy="0 0 0" xyz="0 0 0"/>
+        <geometry>
+          <box size="0.001 0.001 0.001"/>
+        </geometry>
+        <material name="silver"/>
+      </visual>
+      <collision>
+        <origin rpy="0 0 0" xyz="0 0 0"/>
+        <geometry>
+          <box size="0.001 0.001 0.001"/>
+        </geometry>
+      </collision>
+    </link>
+    <joint name="world_joint" type="fixed">
+      <parent link="world"/>
+      <child link="base_link"/>
+      <origin xyz="0 0 0.01" rpy="0 0 0"/>
+    </joint>
+  </xacro:unless>
+  <xacro:if value="${ns == 'left'}">
+    <link name="link_1">
+      <inertial>
+        <origin rpy="0 0 0" xyz="-0.00789643305978462 0.002474313899377526 0.01425764348212194" />
+        <mass value="0.17435766910618158" />
+        <inertia ixx="9.7e-05" ixy="7e-06" ixz="2.8e-05" iyy="0.000111" iyz="-1.2e-05" izz="0.000119" />
+      </inertial>
+      <visual>
+        <origin rpy="0 0 0" xyz="0.003226 0.019004 -0.084836" />
+        <geometry>
+          <mesh filename="package://arm2d2_description/meshes/link1_1.stl" scale="0.001 0.001 0.001" />
+        </geometry>
+        <material name="silver" />
+      </visual>
+      <collision>
+        <origin rpy="0 0 0" xyz="0.003226 0.019004 -0.084836" />
+        <geometry>
+          <mesh filename="package://arm2d2_description/meshes/link1_1.stl" scale="0.001 0.001 0.001" />
+        </geometry>
+      </collision>
+    </link>
+    <joint name="joint_1" type="revolute">
+      <origin rpy="0 0 0" xyz="-0.003226 -0.019004 0.084836" />
+      <parent link="base_link" />
+      <child link="link_1" />
+      <axis xyz="-0.0 -0.0 1.0" />
+      <limit effort="100" lower="-3.1415" upper="3.1415" velocity="100"/>
+    </joint>
+  </xacro:if>
+  <xacro:if value="${ns == 'right'}">
+    <link name="link_1">
+      <inertial>
+        <origin rpy="0 0 0" xyz="0.007896441922670472 0.002474313899377481 0.014257643482122176"/>
+        <mass value="0.17435766910618158"/>
+        <inertia ixx="9.7e-05" ixy="-7e-06" ixz="-2.8e-05" iyy="0.000111" iyz="-1.2e-05" izz="0.000119"/>
+      </inertial>
+      <visual>
+        <origin rpy="0 0 0" xyz="-0.140459 0.019004 -0.084836"/>
+        <geometry>
+          <mesh filename="package://arm2d2_description/meshes/right_link_1.stl" scale="0.001 0.001 0.001"/>
+        </geometry>
+        <material name="silver"/>
+      </visual>
+      <collision>
+        <origin rpy="0 0 0" xyz="-0.140459 0.019004 -0.084836"/>
+        <geometry>
+          <mesh filename="package://arm2d2_description/meshes/right_link_1.stl" scale="0.001 0.001 0.001"/>
+        </geometry>
+      </collision>
+    </link>
+    <joint name="joint_1" type="revolute">
+      <origin rpy="0 0 0" xyz="0.140459 -0.019004 0.084836"/>
+      <parent link="base_link"/>
+      <child link="link_1"/>
+      <axis xyz="-0.0 -0.0 1.0"/>
+      <limit effort="100" lower="-3.1415" upper="3.1415" velocity="100"/>
+    </joint>
+  </xacro:if>
   <link name="link_2">
     <inertial>
@@ -82,5 +118,10 @@
   </link>
   <joint name="joint_2" type="revolute">
-    <origin rpy="0 0 0" xyz="-0.02 0.012069 0.04316" />
+    <xacro:if value="${ns == 'left'}">
+      <origin rpy="0 0 0" xyz="-0.02 0.012069 0.04316" />
+    </xacro:if>
+    <xacro:if value="${ns == 'right'}">
+      <origin rpy="0 0 3.14159" xyz="0.02 0.012069 0.04316" />
+    </xacro:if>
     <parent link="link_1" />
     <child link="link_2" />
@@ -169,87 +210,4 @@
     <limit effort="100" lower="-2.268928" upper="2.268928" velocity="100" />
   </joint>
-  <!--
-  <link name="finger_1">
-    <inertial>
-      <origin rpy="0 0 0" xyz="0.0021645135231446733 0.0056789212234661345 0.027279474187493324" />
-      <mass value="0.005277222771828628" />
-      <inertia ixx="2e-06" ixy="0.0" ixz="0.0" iyy="2e-06" iyz="-0.0" izz="0.0" />
-    </inertial>
-    <visual>
-      <origin rpy="0 0 0" xyz="-0.038503 0.023636 -0.424996" />
-      <geometry>
-        <mesh filename="package://arm2d2_description/meshes/finger_1.stl" scale="0.001 0.001 0.001" />
-      </geometry>
-      <material name="silver" />
-    </visual>
-    <collision>
-      <origin rpy="0 0 0" xyz="-0.038503 0.023636 -0.424996" />
-      <geometry>
-        <mesh filename="package://arm2d2_description/meshes/finger_1.stl" scale="0.001 0.001 0.001" />
-      </geometry>
-    </collision>
-  </link>
-  <joint name="finger_joint1" type="revolute">
-    <origin rpy="0 0 0" xyz="0.041729 -0.016702 0.047" />
-    <parent link="palm" />
-    <child link="finger_1" />
-    <axis xyz="-0.5 -0.866025 6e-06" />
-    <limit effort="100" lower="-0.698132" upper="0.0" velocity="100" />
-  </joint>
-  <link name="finger_2">
-    <inertial>
-      <origin rpy="0 0 0" xyz="-0.0021646025973648094 0.00567892122346535 0.027279474187493602" />
-      <mass value="0.005277222771828628" />
-      <inertia ixx="2e-06" ixy="-0.0" ixz="-0.0" iyy="2e-06" iyz="-0.0" izz="0.0" />
-    </inertial>
-    <visual>
-      <origin rpy="0 0 0" xyz="-0.005046 0.023636 -0.424996" />
-      <geometry>
-        <mesh filename="package://arm2d2_description/meshes/finger_2.stl" scale="0.001 0.001 0.001" />
-      </geometry>
-      <material name="silver" />
-    </visual>
-    <collision>
-      <origin rpy="0 0 0" xyz="-0.005046 0.023636 -0.424996" />
-      <geometry>
-        <mesh filename="package://arm2d2_description/meshes/finger_2.stl" scale="0.001 0.001 0.001" />
-      </geometry>
-    </collision>
-  </link>
-  <joint name="finger_joint2" type="revolute">
-    <origin rpy="0 0 0" xyz="0.008272 -0.016702 0.047" />
-    <parent link="palm" />
-    <child link="finger_2" />
-    <axis xyz="0.5 -0.866025 6e-06" />
-    <limit effort="100" lower="0.0" upper="0.698132" velocity="100" />
-  </joint>
-  <link name="finger_3">
-    <inertial>
-      <origin rpy="0 0 0" xyz="0.006000455462889673 -0.000964137225942182 0.02727923439293578" />
-      <mass value="0.005277222771828628" />
-      <inertia ixx="2e-06" ixy="0.0" ixz="0.0" iyy="2e-06" iyz="0.0" izz="0.0" />
-    </inertial>
-    <visual>
-      <origin rpy="0 0 0" xyz="-0.015674 -0.015904 -0.424996" />
-      <geometry>
-        <mesh filename="package://arm2d2_description/meshes/finger_3.stl" scale="0.001 0.001 0.001" />
-      </geometry>
-      <material name="silver" />
-    </visual>
-    <collision>
-      <origin rpy="0 0 0" xyz="-0.015674 -0.015904 -0.424996" />
-      <geometry>
-        <mesh filename="package://arm2d2_description/meshes/finger_3.stl" scale="0.001 0.001 0.001" />
-      </geometry>
-    </collision>
-  </link>
-  <joint name="finger_joint3" type="revolute">
-    <origin rpy="0 0 0" xyz="0.0189 0.022838 0.047" />
-    <parent link="palm" />
-    <child link="finger_3" />
-    <axis xyz="-1.0 0.0 -0.0" />
-    <limit effort="100" lower="0.0" upper="0.698132" velocity="100" />
-  </joint>
-  -->
   <transmission name="transmission_1">
     <type>transmission_interface/SimpleTransmission</type>
@@ -302,36 +260,4 @@
     </actuator>
   </transmission>
-  <!--
-  <transmission name="trans_finger_joint1">
-    <type>transmission_interface/SimpleTransmission</type>
-    <joint name="finger_joint1">
-      <hardwareInterface>hardware_interface/PositionJointInterface</hardwareInterface>
-    </joint>
-    <actuator name="finger_joint1_motor">
-      <hardwareInterface>hardware_interface/PositionJointInterface</hardwareInterface>
-      <mechanicalReduction>1</mechanicalReduction>
-    </actuator>
-  </transmission>
-  <transmission name="trans_finger_joint2">
-    <type>transmission_interface/SimpleTransmission</type>
-    <joint name="finger_joint2">
-      <hardwareInterface>hardware_interface/PositionJointInterface</hardwareInterface>
-    </joint>
-    <actuator name="finger_joint2_motor">
-      <hardwareInterface>hardware_interface/PositionJointInterface</hardwareInterface>
-      <mechanicalReduction>1</mechanicalReduction>
-    </actuator>
-  </transmission>
-  <transmission name="trans_finger_joint3">
-    <type>transmission_interface/SimpleTransmission</type>
-    <joint name="finger_joint3">
-      <hardwareInterface>hardware_interface/PositionJointInterface</hardwareInterface>
-    </joint>
-    <actuator name="finger_joint3_motor">
-      <hardwareInterface>hardware_interface/PositionJointInterface</hardwareInterface>
-      <mechanicalReduction>1</mechanicalReduction>
-    </actuator>
-  </transmission>
-  -->
   <gazebo>
     <plugin name="gazebo_ros_control" filename="libgazebo_ros_control.so">
@@ -376,23 +302,3 @@
     <selfCollide>true</selfCollide>
   </gazebo>
-  <!--
-  <gazebo reference="finger_1">
-    <material>Gazebo/Silver</material>
-    <mu1>0.2</mu1>
-    <mu2>0.2</mu2>
-    <selfCollide>true</selfCollide>
-  </gazebo>
-  <gazebo reference="finger_2">
-    <material>Gazebo/Silver</material>
-    <mu1>0.2</mu1>
-    <mu2>0.2</mu2>
-    <selfCollide>true</selfCollide>
-  </gazebo>
-  <gazebo reference="finger_3">
-    <material>Gazebo/Silver</material>
-    <mu1>0.2</mu1>
-    <mu2>0.2</mu2>
-    <selfCollide>true</selfCollide>
-  </gazebo>
-  -->
 </robot>

File: arm2d2/arm2d2_description/urdf/arm2d2.xacro (robot description, xacro)
@@ -4,4 +4,6 @@
   <xacro:arg name="include_arm" default="false"/>
   <xacro:arg name="include_gripper" default="false"/>
+  <!-- When true each arm comes with the base attached (always false in this file)-->
+  <xacro:arg name="include_arm_base" default="false"/>
   <!-- Convert args to properties-->
   <xacro:property name="ns" value="$(arg ns)"/>
@@ -27,8 +29,8 @@
         <child link="gripper_link"/>
         <xacro:if value="${is_left}">
-          <origin xyz="0.025 0 0.025" rpy="0 0 0"/>
+          <origin xyz="0.025 0 0.009" rpy="0 0 0"/>
         </xacro:if>
         <xacro:unless value="${is_left}">
-          <origin xyz="0.025 0 0.025" rpy="0 0 3.14159"/>
+          <origin xyz="0.025 0 0.009" rpy="0 0 3.14159"/>
         </xacro:unless>
       </joint>

File: arm2d2/arm2d2_description/urdf/base.urdf.xacro (robot description, xacro)
@@ -2,4 +2,5 @@
 <robot name="arm2d" xmlns:xacro="http://www.ros.org/wiki/xacro">
 <xacro:arg name="top_plate" default="false"/>
+<link name="world"/>
 <link name="base_link">
   <inertial>
@@ -22,4 +23,9 @@
   </collision>
 </link>
+<joint name="world_joint" type="fixed">
+  <origin xyz="0 0 0" rpy="0 0 0"/>
+  <parent link="world"/>
+  <child link="base_link"/>
+</joint>
 <xacro:if value="$(arg top_plate)">
   <link name="top_plate">

Commit message: First round of removing complete

File: arm2d2/arm2d2_description/urdf/arm1_gazebo.urdf.xacro (robot description, xacro)
@@ -49,5 +49,5 @@
         <origin rpy="0 0 0" xyz="0.003226 0.019004 -0.084836" />
         <geometry>
-          <mesh filename="package://arm2d2_description/meshes/link1_1.stl" scale="0.001 0.001 0.001" />
+          <mesh filename="package://arm2d2_description/meshes/link_1.stl" scale="0.001 0.001 0.001" />
         </geometry>
         <material name="silver" />
@@ -56,5 +56,5 @@
         <origin rpy="0 0 0" xyz="0.003226 0.019004 -0.084836" />
         <geometry>
-          <mesh filename="package://arm2d2_description/meshes/link1_1.stl" scale="0.001 0.001 0.001" />
+          <mesh filename="package://arm2d2_description/meshes/link_1.stl" scale="0.001 0.001 0.001" />
         </geometry>
       </collision>
@@ -106,5 +106,5 @@
       <origin rpy="0 0 0" xyz="0.023226 0.006935 -0.127996" />
       <geometry>
-        <mesh filename="package://arm2d2_description/meshes/link2_1.stl" scale="0.001 0.001 0.001" />
+        <mesh filename="package://arm2d2_description/meshes/link_2.stl" scale="0.001 0.001 0.001" />
       </geometry>
       <material name="silver" />
@@ -113,5 +113,5 @@
       <origin rpy="0 0 0" xyz="0.023226 0.006935 -0.127996" />
       <geometry>
-        <mesh filename="package://arm2d2_description/meshes/link2_1.stl" scale="0.001 0.001 0.001" />
+        <mesh filename="package://arm2d2_description/meshes/link_2.stl" scale="0.001 0.001 0.001" />
       </geometry>
     </collision>
@@ -138,5 +138,5 @@
       <origin rpy="0 0 0" xyz="0.013226 0.006935 -0.247996" />
       <geometry>
-        <mesh filename="package://arm2d2_description/meshes/link3_1.stl" scale="0.001 0.001 0.001" />
+        <mesh filename="package://arm2d2_description/meshes/link_3.stl" scale="0.001 0.001 0.001" />
       </geometry>
       <material name="silver" />
@@ -145,5 +145,5 @@
       <origin rpy="0 0 0" xyz="0.013226 0.006935 -0.247996" />
       <geometry>
-        <mesh filename="package://arm2d2_description/meshes/link3_1.stl" scale="0.001 0.001 0.001" />
+        <mesh filename="package://arm2d2_description/meshes/link_3.stl" scale="0.001 0.001 0.001" />
       </geometry>
     </collision>
@@ -165,5 +165,5 @@
       <origin rpy="0 0 0" xyz="-0.006774 0.006935 -0.287996" />
       <geometry>
-        <mesh filename="package://arm2d2_description/meshes/link4_1.stl" scale="0.001 0.001 0.001" />
+        <mesh filename="package://arm2d2_description/meshes/link_4.stl" scale="0.001 0.001 0.001" />
       </geometry>
       <material name="silver" />
@@ -172,5 +172,5 @@
       <origin rpy="0 0 0" xyz="-0.006774 0.006935 -0.287996" />
       <geometry>
-        <mesh filename="package://arm2d2_description/meshes/link4_1.stl" scale="0.001 0.001 0.001" />
+        <mesh filename="package://arm2d2_description/meshes/link_4.stl" scale="0.001 0.001 0.001" />
       </geometry>
     </collision>
@@ -272,29 +272,29 @@
     <gravity>true</gravity>
   </gazebo>
-  <gazebo reference="link1">
-    <material>Gazebo/Silver</material>
-    <mu1>0.2</mu1>
-    <mu2>0.2</mu2>
-    <selfCollide>true</selfCollide>
-  </gazebo>
-  <gazebo reference="link2">
-    <material>Gazebo/Silver</material>
-    <mu1>0.2</mu1>
-    <mu2>0.2</mu2>
-    <selfCollide>true</selfCollide>
-  </gazebo>
-  <gazebo reference="link3">
-    <material>Gazebo/Silver</material>
-    <mu1>0.2</mu1>
-    <mu2>0.2</mu2>
-    <selfCollide>true</selfCollide>
-  </gazebo>
-  <gazebo reference="link4">
-    <material>Gazebo/Silver</material>
-    <mu1>0.2</mu1>
-    <mu2>0.2</mu2>
-    <selfCollide>true</selfCollide>
-  </gazebo>
-  <gazebo reference="palm">
+  <gazebo reference="link_1">
+    <material>Gazebo/Silver</material>
+    <mu1>0.2</mu1>
+    <mu2>0.2</mu2>
+    <selfCollide>true</selfCollide>
+  </gazebo>
+  <gazebo reference="link_2">
+    <material>Gazebo/Silver</material>
+    <mu1>0.2</mu1>
+    <mu2>0.2</mu2>
+    <selfCollide>true</selfCollide>
+  </gazebo>
+  <gazebo reference="link_3">
+    <material>Gazebo/Silver</material>
+    <mu1>0.2</mu1>
+    <mu2>0.2</mu2>
+    <selfCollide>true</selfCollide>
+  </gazebo>
+  <gazebo reference="link_4">
+    <material>Gazebo/Silver</material>
+    <mu1>0.2</mu1>
+    <mu2>0.2</mu2>
+    <selfCollide>true</selfCollide>
+  </gazebo>
+  <gazebo reference="link_5">
     <material>Gazebo/Silver</material>
     <mu1>0.2</mu1>

Commit message: Fixed launching with base

File: arm2d2/arm2d2_description/urdf/arm1_gazebo.urdf.xacro (robot description, xacro)
@@ -3,4 +3,5 @@
   <xacro:arg name="include_arm_base" default="true"/>
   <xacro:arg name="ns" default="left"/>
+  <xacro:arg name="include_gripper" default="false"/>
   <!-- Convert arg to property -->
   <xacro:property name="ns" value="$(arg ns)"/>
@@ -210,4 +211,40 @@
     <limit effort="100" lower="-2.268928" upper="2.268928" velocity="100" />
   </joint>
+  <!-- Fake link that allows gripper to "spin" even though the hardware does not have a revolute gripper joint -->
+  <xacro:if value="$(arg include_gripper)">
+    <link name="gripper_connector">
+      <inertial>
+        <origin rpy="0 0 0" xyz="2.9287E-10 -1.6472E-09 0.0091432"/>
+        <mass value="0.013863"/>
+        <inertia ixx="1.3596E-06" ixy="3.0585E-13" ixz="5.7102E-14" iyy="1.7157E-06" iyz="6.3369E-09" izz="2.4332E-06"/>
+      </inertial>
+    </link>
+  </xacro:if>
+  <!-- Box that provides gripper collider only for moveit so gazebo does not simulate collisions -->
+  <xacro:unless value="$(arg include_gripper)">
+    <link name="gripper_connector">
+      <xacro:unless value="$(arg include_gripper)">
+        <collision>
+          <origin xyz="0.025 0 0.075" rpy="0 0 0" />
+          <geometry>
+            <box size="0.05 0.05 0.05"/>
+          </geometry>
+        </collision>
+      </xacro:unless>
+      <visual>
+        <origin xyz="0.025 0 0.075" rpy="0 0 0" />
+        <geometry>
+          <box size="0.05 0.05 0.05"/>
+        </geometry>
+      </visual>
+    </link>
+  </xacro:unless>
+  <joint name="gripper_joint" type="revolute">
+    <origin xyz="0 0 0" rpy="0 0 0" />
+    <parent link="link_5"/>
+    <child link="gripper_connector"/>
+    <axis xyz="0 0 1"/>
+    <limit lower="-3.1415" upper="3.1415" effort="100" velocity="100"/>
+  </joint>
   <transmission name="transmission_1">
     <type>transmission_interface/SimpleTransmission</type>
@@ -256,4 +293,14 @@
     </joint>
     <actuator name="motor_5">
+      <hardwareInterface>hardware_interface/PositionJointInterface</hardwareInterface>
+      <mechanicalReduction>1</mechanicalReduction>
+    </actuator>
+  </transmission>
+  <transmission name="transmission_6">
+    <type>transmission_interface/SimpleTransmission</type>
+    <joint name="gripper_joint">
+      <hardwareInterface>hardware_interface/PositionJointInterface</hardwareInterface>
+    </joint>
+    <actuator name="motor_6">
       <hardwareInterface>hardware_interface/PositionJointInterface</hardwareInterface>
       <mechanicalReduction>1</mechanicalReduction>
@@ -302,3 +349,9 @@
     <selfCollide>true</selfCollide>
   </gazebo>
+  <gazebo reference="gripper_joint">
+    <material>Gazebo/Silver</material>
+    <mu1>0.2</mu1>
+    <mu2>0.2</mu2>
+    <selfCollide>true</selfCollide>
+  </gazebo>
 </robot>

File: arm2d2/arm2d2_description/urdf/arm2d2.xacro (robot description, xacro)
@@ -25,5 +25,5 @@
   <xacro:if value="$(arg include_arm)">
     <xacro:if value="$(arg include_gripper)">
-      <joint name="gripper_joint" type="fixed">
+      <joint name="gripper_connect_joint" type="fixed">
         <parent link="link_5"/>
         <child link="gripper_link"/>
