Commit message: Updated models

File: arm2d2/arm2d2_description/urdf/base.urdf.xacro (robot description, xacro)
@@ -2,4 +2,9 @@
 <robot name="arm2d" xmlns:xacro="http://www.ros.org/wiki/xacro">
 <xacro:arg name="top_plate" default="false"/>
+<xacro:property name="long_l" value="0.02"/>
+<xacro:property name="long_w" value="0.05"/>
+<xacro:property name="long_h" value="0.279654"/>
+<link name="world"/>
+<!--
 <link name="base_link">
   <inertial>
@@ -11,5 +16,5 @@
     <origin rpy="0 0 0" xyz="0 0 0"/>
     <geometry>
-      <mesh filename="package://arm2d2_description/meshes/base_link.stl" scale="0.001 0.001 0.001"/>
+      <mesh filename="package://arm2d2_description/meshes/base_plate.stl" scale="0.001 0.001 0.001"/>
     </geometry>
     <material name="silver"/>
@@ -18,8 +23,149 @@
     <origin rpy="0 0 0" xyz="0 0 0"/>
     <geometry>
-      <mesh filename="package://arm2d2_description/meshes/base_link.stl" scale="0.001 0.001 0.001"/>
+      <mesh filename="package://arm2d2_description/meshes/base_plate.stl" scale="0.001 0.001 0.001"/>
     </geometry>
   </collision>
 </link>
+-->
+<link name="base_link">
+  <inertial>
+    <origin xyz="-2.154281413321998e-06 0.0035387814754625734 -0.0056639470834143136" rpy="0 0 0"/>
+    <mass value="1.5479093566761954"/>
+    <inertia ixx="0.010238" iyy="0.01139" izz="0.021617" ixy="-0.0" iyz="0.0" ixz="0.0"/>
+  </inertial>
+  <visual>
+    <origin xyz="0 0 0.0025" rpy="0 0 0"/>
+    <geometry>
+      <mesh filename="package://arm2d2_description/meshes/base_plate.stl" scale="0.001 0.001 0.001"/>
+    </geometry>
+    <material name="silver"/>
+  </visual>
+  <collision>
+    <origin xyz="0 0 0.0025" rpy="0 0 0"/>
+    <geometry>
+      <mesh filename="package://arm2d2_description/meshes/base_plate.stl" scale="0.001 0.001 0.001"/>
+    </geometry>
+  </collision>
+</link>
+<joint name="world_joint" type="fixed">
+  <origin xyz="0 0.0025 0.078232" rpy="0 0 0"/>
+  <parent link="world"/>
+  <child link="base_link"/>
+</joint>
+<link name="gripper_mount_l">
+  <inertial>
+    <origin xyz="0.060099999999972134 -0.08246115124410087 0.038698562774923354" rpy="0 0 0"/>
+    <mass value="0.06861748378285525"/>
+    <inertia ixx="1.9e-05" iyy="1.9e-05" izz="1.7e-05" ixy="0.0" iyz="0.0" ixz="-0.0"/>
+  </inertial>
+  <visual>
+    <origin xyz="-0.0 3e-06 0.011329" rpy="0 0 0"/>
+    <geometry>
+      <mesh filename="package://arm2d2_description/meshes/gripper_mount.stl" scale="0.001 0.001 0.001"/>
+    </geometry>
+    <material name="silver"/>
+  </visual>
+  <!--<collision>
+    <origin xyz="-0.0 3e-06 0.011329" rpy="0 0 0"/>
+    <geometry>
+      <mesh filename="package://arm2d2_description/meshes/gripper_mount.stl" scale="0.001 0.001 0.001"/>
+    </geometry>
+  </collision>-->
+</link>
+<joint name="gripper_mount_l_joint" type="fixed">
+  <origin xyz="-0.12 -3e-06 -0.008829" rpy="0 0 0"/>
+  <parent link="base_link"/>
+  <child link="gripper_mount_l"/>
+</joint>
+<link name="gripper_mount_r">
+  <inertial>
+    <origin xyz="0.060099999999972134 -0.08246115124410087 0.038698562774923354" rpy="0 0 0"/>
+    <mass value="0.06861748378285525"/>
+    <inertia ixx="1.9e-05" iyy="1.9e-05" izz="1.7e-05" ixy="0.0" iyz="0.0" ixz="-0.0"/>
+  </inertial>
+  <visual>
+    <origin xyz="-0.0 3e-06 0.011329" rpy="0 0 0"/>
+    <geometry>
+      <mesh filename="package://arm2d2_description/meshes/gripper_mount.stl" scale="0.001 0.001 0.001"/>
+    </geometry>
+    <material name="silver"/>
+  </visual>
+  <!--<collision>
+    <origin xyz="-0.0 3e-06 0.011329" rpy="0 0 0"/>
+    <geometry>
+      <mesh filename="package://arm2d2_description/meshes/gripper_mount.stl" scale="0.001 0.001 0.001"/>
+    </geometry>
+  </collision>-->
+</link>
+<joint name="gripper_mount_r_joint" type="fixed">
+  <origin xyz="0 -3e-06 -0.008829" rpy="0 0 0"/>
+  <parent link="base_link"/>
+  <child link="gripper_mount_r"/>
+</joint>
+<link name="soft_robotics">
+  <visual>
+    <origin xyz="0 -0.04184 0.063" rpy="0 0 0"/>
+    <geometry>
+      <box size="0.05 0.15 0.125"/>
+    </geometry>
+  </visual>
+</link>
+<joint name="srob_joint" type="fixed">
+  <origin xyz="0 0 0" rpy="0 0 0"/>
+  <parent link="base_link"/>
+  <child link="soft_robotics"/>
+</joint>
+<link name="longeron_1">
+  <visual>
+    <origin xyz="0 0 0" rpy="0 0 0"/>
+    <geometry>
+      <box size="${long_l} ${long_w} ${long_h}"/>
+    </geometry>
+  </visual>
+</link>
+<joint name="longeron_1_j" type="fixed">
+  <origin xyz="0.175 0 0.0616" rpy="0 0 0"/>
+  <parent link="base_link"/>
+  <child link="longeron_1"/>
+</joint>
+<link name="longeron_2">
+  <visual>
+    <origin xyz="0 0 0" rpy="0 0 0"/>
+    <geometry>
+      <box size="${long_l} ${long_w} ${long_h}"/>
+    </geometry>
+  </visual>
+</link>
+<joint name="longeron_2_j" type="fixed">
+  <origin xyz="-0.175 0 0.0616" rpy="0 0 0"/>
+  <parent link="base_link"/>
+  <child link="longeron_2"/>
+</joint>
+<link name="longeron_3">
+  <visual>
+    <origin xyz="0 0 0" rpy="0 0 0"/>
+    <geometry>
+      <box size="${long_w} ${long_l} ${long_h}"/>
+    </geometry>
+  </visual>
+</link>
+<joint name="longeron_3_j" type="fixed">
+  <origin xyz="0 0.1725 0.0616" rpy="0 0 0"/>
+  <parent link="base_link"/>
+  <child link="longeron_3"/>
+</joint>
+<link name="longeron_4">
+  <visual>
+    <origin xyz="0 0 0" rpy="0 0 0"/>
+    <geometry>
+      <box size="${long_w} ${long_l} ${long_h}"/>
+    </geometry>
+  </visual>
+</link>
+<joint name="longeron_4_j" type="fixed">
+  <origin xyz="0 -0.1725 0.0616" rpy="0 0 0"/>
+  <parent link="base_link"/>
+  <child link="longeron_4"/>
+</joint>
 <xacro:if value="$(arg top_plate)">
   <link name="top_plate">
@@ -44,5 +190,5 @@
   </link>
   <joint name="top_plate_joint" type="fixed">
-    <origin rpy="0 0 0" xyz="0.068617 -0.090846 0.29"/>
+    <origin rpy="0 0 0" xyz="0.068617 -0.090846 0.204724"/>
     <parent link="base_link"/>
     <child link="top_plate"/>

Commit message: Two updated simulated arms can fold

File: arm2d2/arm2d2_description/urdf/arm1_gazebo.urdf.xacro (robot description, xacro)
@@ -15,6 +15,14 @@
   <xacro:unless value="$(arg include_arm_base)">
     <link name="world"/>
-  <link name="base_link">
-    <inertial>
+    <link name="base_link"/>
+    <joint name="world_joint" type="fixed">
+      <parent link="world"/>
+      <child link="base_link"/>
+      <!-- rpy="1.57 0 0"-->
+      <origin xyz="0 0 0.0775" rpy="0 0 0"/>
+    </joint>
+  </xacro:unless>
+  <link name="base_connector">
+      <inertial>
       <origin rpy="0 0 0" xyz="0.06861790086338357 -0.0835697992386399 0.07107579694115096"/>
       <mass value="4.519107238213137"/>
@@ -35,39 +43,42 @@
     </collision>
   </link>
-    <joint name="world_joint" type="fixed">
-      <parent link="world"/>
-      <child link="base_link"/>
-      <origin xyz="0 0 0.0725" rpy="1.57 0 0"/>
-    </joint>
-  </xacro:unless>
-  <xacro:if value="${ns == 'left'}">
-    <link name="link_1">
-      <inertial>
-        <origin xyz="-0.023234210000508494 0.032933361084236216 0.002920663644532681" rpy="0 0 0"/>
-        <mass value="0.22666453646044638"/>
-        <inertia ixx="0.000128" iyy="0.000201" izz="0.000231" ixy="3.1e-05" iyz="-5e-06" ixz="1.5e-05"/>
-      </inertial>
-      <visual>
-        <origin xyz="-0.0851 -0.006604 0.0851" rpy="0 0 0"/>
-        <geometry>
-          <mesh filename="package://arm2d2_description/meshes/link_1_1.stl" scale="0.001 0.001 0.001"/>
-        </geometry>
-        <material name="silver"/>
-      </visual>
-      <collision>
-        <origin xyz="-0.0851 -0.006604 0.0851" rpy="0 0 0"/>
-        <geometry>
-          <mesh filename="package://arm2d2_description/meshes/link_1_1.stl" scale="0.001 0.001 0.001"/>
-        </geometry>
-      </collision>
-    </link>
-    <joint name="joint_1" type="revolute">
-      <origin xyz="0.0851 0.006604 -0.0851" rpy="0 0 0"/>
-      <parent link="base_link"/>
-      <child link="link_1"/>
-      <axis xyz="0.0 -1.0 0.0"/>
-      <limit effort="100" lower="-3.1415" upper="3.1415" velocity="100"/>
-    </joint>
-  </xacro:if>
+  <joint name="base_connector_joint" type="fixed">
+    <parent link="base_link"/>
+    <child link="base_connector"/>
+    <origin xyz="0 0 -0.005" rpy="1.57 0 0"/>
+  </joint>
+  <link name="link_1">
+    <inertial>
+      <origin xyz="-0.023234210000508494 0.032933361084236216 0.002920663644532681" rpy="0 0 0"/>
+      <mass value="0.22666453646044638"/>
+      <inertia ixx="0.000128" iyy="0.000201" izz="0.000231" ixy="3.1e-05" iyz="-5e-06" ixz="1.5e-05"/>
+    </inertial>
+    <visual>
+      <origin xyz="-0.0851 -0.006604 0.0851" rpy="0 0 0"/>
+      <geometry>
+        <mesh filename="package://arm2d2_description/meshes/link_1_1.stl" scale="0.001 0.001 0.001"/>
+      </geometry>
+      <material name="silver"/>
+    </visual>
+    <collision>
+      <origin xyz="-0.0851 -0.006604 0.0851" rpy="0 0 0"/>
+      <geometry>
+        <mesh filename="package://arm2d2_description/meshes/link_1_1.stl" scale="0.001 0.001 0.001"/>
+      </geometry>
+    </collision>
+  </link>
+  <joint name="joint_1" type="revolute">
+    <!-- p value corresponds to starting point for stepper -->
+    <xacro:if value="${ns == 'left'}">
+      <origin xyz="-0.0851 0.006604 -0.0851" rpy="0 2.82584 0"/>
+    </xacro:if>
+    <xacro:unless value="${ns == 'left'}">
+      <origin xyz="0.0851 0.006604 -0.0851" rpy="0 0.15708 0"/>
+    </xacro:unless>
+    <parent link="base_connector"/>
+    <child link="link_1"/>
+    <axis xyz="0.0 -1.0 0.0"/>
+    <limit effort="100" lower="-3.1415" upper="3.1415" velocity="100"/>
+  </joint>
   <link name="link_2">
     <inertial>
@@ -92,10 +103,14 @@
   <joint name="joint_2" type="revolute">
     <xacro:if value="${ns == 'left'}">
+      <origin xyz="0.005205 0.04 -0.000685" rpy="-0.436332 0 0.03927"/>
+      <limit lower="-1.919862" upper="1.396263" effort="100" velocity="100"/>
+    </xacro:if>
+    <xacro:unless value="${ns == 'left'}">
       <origin xyz="0.005205 0.04 -0.000685" rpy="0 0 0"/>
-    </xacro:if>
+      <limit upper="1.919862" lower="-1.396263" effort="100" velocity="100"/>
+    </xacro:unless>
     <parent link="link_1" />
     <child link="link_2" />
     <axis xyz="-0.991445 -0.0 0.130526"/>
-    <limit upper="1.919862" lower="-1.396263" effort="100" velocity="100"/>
   </joint>
   <link name="link_3">
@@ -120,9 +135,15 @@
   </link>
   <joint name="joint_3" type="revolute">
-    <origin xyz="-0.005959 0.136681 0.031347" rpy="0 0 0"/>
+    <xacro:if value="${ns == 'left'}">
+     <origin xyz="-0.005959 0.136681 0.031347" rpy="-3.42078 0.23562 -0.03"/>
+     <limit lower="-4.101524" upper="0.698132" effort="100" velocity="100"/>
+    </xacro:if>
+    <xacro:unless value="${ns == 'left'}">
+      <origin xyz="-0.005959 0.136681 0.031347" rpy="0 0 0"/>
+      <limit upper="4.101524" lower="-0.698132" effort="100" velocity="100"/>
+    </xacro:unless>
     <parent link="link_2" />
     <child link="link_3" />
     <axis xyz="-0.991445 -0.0 0.130526"/>
-    <limit upper="4.101524" lower="-0.698132" effort="100" velocity="100"/>
   </joint>
   <link name="link_4">
@@ -174,9 +195,15 @@
   </link>
   <joint name="joint_5" type="revolute">
-    <origin xyz="0.032067 -0.036743 0.089586" rpy="0 0 0"/>
+    <xacro:if value="${ns == 'left'}">
+     <origin xyz="0.032067 -0.036743 0.089586" rpy="-2.38412 0.23562 0.1"/>
+     <limit lower="-3.228859" upper="0.785398" effort="100" velocity="100"/>
+    </xacro:if>
+    <xacro:unless value="${ns == 'left'}">
+      <origin xyz="0.032067 -0.036743 0.089586" rpy="0 0 0"/>
+      <limit upper="3.228859" lower="-0.785398" effort="100" velocity="100"/>
+    </xacro:unless>
     <parent link="link_4" />
     <child link="link_5" />
     <axis xyz="-0.991445 -0.0 0.130526"/>
-    <limit upper="3.228859" lower="-0.785398" effort="100" velocity="100"/>
   </joint>
   <!-- Fake link that allows gripper to "spin" even though the hardware does not have a revolute gripper joint -->
@@ -193,4 +220,11 @@
   <xacro:unless value="$(arg include_gripper)">
     <link name="gripper_connector">
+      <inertial>
+        <origin rpy="0 0 0" xyz="2.9287E-10 -1.6472E-09 0.0091432"/>
+        <mass value="0.013863"/>
+        <inertia ixx="1.3596E-06" ixy="3.0585E-13" ixz="5.7102E-14" iyy="1.7157E-06" iyz="6.3369E-09" izz="2.4332E-06"/>
+      </inertial>
+    </link>
+    <link name="gripper_collider">
       <xacro:unless value="$(arg include_gripper)">
         <!-- Removed to test sim handoff
@@ -211,7 +245,12 @@
       </visual>-->
     </link>
+    <joint name="gripper_collider_joint" type="fixed">
+      <origin xyz="0 0 0" rpy="0 0 0"/>
+      <parent link="link_5"/>
+      <child link="gripper_collider"/>
+    </joint>
   </xacro:unless>
   <joint name="gripper_joint" type="revolute">
-    <origin xyz="0 0 0" rpy="0 0 0" />
+    <origin xyz="-0.03 -0.041 0.0045" rpy="0 0 0"/>
     <parent link="link_5"/>
     <child link="gripper_connector"/>

File: arm2d2/arm2d2_description/urdf/arm2d2.xacro (robot description, xacro)
@@ -31,8 +31,10 @@
         <xacro:if value="${is_left}">
           <!-- Very wierd axis because link_5 is upside down (x, z, y)-->
+          <!-- <origin xyz="-0.03 -0.041 0.0045" rpy="0 0 0"/> -->
           <origin xyz="-0.03 -0.041 0.0045" rpy="0 0 0"/>
         </xacro:if>
         <xacro:unless value="${is_left}">
-          <origin xyz="0.025 0 0.009" rpy="0 0 3.14159"/>
+          <!-- <origin xyz="0.025 0 0.009" rpy="0 0 3.14159"/> -->
+          <origin xyz="-0.03 -0.041 0.0045" rpy="0 0 0"/>
         </xacro:unless>
       </joint>

File: arm2d2/arm2d2_description/urdf/base.urdf.xacro (robot description, xacro)
@@ -74,5 +74,5 @@
 </link>
 <joint name="gripper_mount_l_joint" type="fixed">
-  <origin xyz="-0.12 -3e-06 -0.008829" rpy="0 0 0"/>
+  <origin xyz="-0.145 -8e-06 -0.008829" rpy="0 0 0"/>
   <parent link="base_link"/>
   <child link="gripper_mount_l"/>
@@ -99,5 +99,5 @@
 </link>
 <joint name="gripper_mount_r_joint" type="fixed">
-  <origin xyz="0 -3e-06 -0.008829" rpy="0 0 0"/>
+  <origin xyz="0.025 -8e-06 -0.008829" rpy="0 0 0"/>
   <parent link="base_link"/>
   <child link="gripper_mount_r"/>
@@ -105,14 +105,30 @@
 <link name="soft_robotics">
   <visual>
-    <origin xyz="0 -0.04184 0.063" rpy="0 0 0"/>
-    <geometry>
-      <box size="0.05 0.15 0.125"/>
+    <origin xyz="0 0 0" rpy="1.57 0 0"/>
+    <geometry>
+      <!-- height is 0.125-->
+      <mesh filename="package://arm2d2_description/meshes/soft_robotics.stl" scale="0.001 0.001 0.001"/>
     </geometry>
   </visual>
 </link>
 <joint name="srob_joint" type="fixed">
+  <origin xyz="-0.03561 0.041939 0" rpy="0 0 0"/>
+  <parent link="base_link"/>
+  <child link="soft_robotics"/>
+</joint>
+<link name="camera_mount">
+  <visual>
+    <!-- z= 0.078232 - 0.01555 + 0.06985 - 0.005 = 0.100711-->
+    <!-- middle of bp - dist to mount hole + dist between longeron holes - dist to mid of mount-->
+    <origin xyz="0.0612 0.165 0.095" rpy="1.57 0 -1.57"/>
+    <geometry>
+      <mesh filename="package://arm2d2_description/meshes/camera_mount.stl" scale="0.001 0.001 0.001"/>
+    </geometry>
+  </visual>
+</link>
+<joint name="cam_joint" type="fixed">
   <origin xyz="0 0 0" rpy="0 0 0"/>
   <parent link="base_link"/>
-  <child link="soft_robotics"/>
+  <child link="camera_mount"/>
 </joint>
 <link name="longeron_1">
@@ -164,5 +180,5 @@
 </link>
 <joint name="longeron_4_j" type="fixed">
-  <origin xyz="0 -0.1725 0.0616" rpy="0 0 0"/>
+  <origin xyz="0 -0.1775 0.0616" rpy="0 0 0"/>
   <parent link="base_link"/>
   <child link="longeron_4"/>
@@ -182,4 +198,5 @@
       <material name="silver"/>
     </visual>
+    <!--
     <collision>
       <origin rpy="0 0 0" xyz="-0.068617 0.090846 -0.0"/>
@@ -188,7 +205,8 @@
       </geometry>
     </collision>
+    -->
   </link>
   <joint name="top_plate_joint" type="fixed">
-    <origin rpy="0 0 0" xyz="0.068617 -0.090846 0.204724"/>
+    <origin rpy="0 0 0" xyz="0.068617 -0.090846 0.211324"/>
     <parent link="base_link"/>
     <child link="top_plate"/>

Commit message: Both arms pickup with state machine

File: arm2d2/arm2d2_description/urdf/arm1_gazebo.urdf.xacro (robot description, xacro)
@@ -71,5 +71,6 @@
     <!-- p value corresponds to starting point for stepper -->
     <xacro:if value="${ns == 'left'}">
-      <origin xyz="-0.0851 0.006604 -0.0851" rpy="0 2.82584 0"/>
+      <!-- p=2.82584 -->
+      <origin xyz="-0.0851 0.006604 -0.0851" rpy="0 2.775 0"/>
     </xacro:if>
     <xacro:unless value="${ns == 'left'}">

File: arm2d2/arm2d2_description/urdf/base.urdf.xacro (robot description, xacro)
@@ -107,5 +107,4 @@
     <origin xyz="0 0 0" rpy="1.57 0 0"/>
     <geometry>
-      <!-- height is 0.125-->
       <mesh filename="package://arm2d2_description/meshes/soft_robotics.stl" scale="0.001 0.001 0.001"/>
     </geometry>
