Commit message: Added unfolding capability

File: arm2d2/arm2d2_description/urdf/base.urdf.xacro (robot description, xacro)
@@ -24,5 +24,5 @@
 </link>
 <joint name="world_joint" type="fixed">
-  <origin xyz="0 0 0" rpy="0 0 0"/>
+  <origin xyz="0 0 0.0075" rpy="0 0 0"/>
   <parent link="world"/>
   <child link="base_link"/>

Commit message: Integrated throw at intervals

File: arm2d2/arm2d2_description/urdf/base.urdf.xacro (robot description, xacro)
@@ -211,5 +211,5 @@
   </link>
   <joint name="top_plate_joint" type="fixed">
-    <origin rpy="0 0 0" xyz="0.068617 -0.090846 0.211324"/>
+    <origin rpy="0 0 0" xyz="0.068617 -0.090846 0.215"/>
     <parent link="base_link"/>
     <child link="top_plate"/>

File: tundra_gripper/urdf/gripper.urdf.xacro (robot description, xacro)
@@ -31,5 +31,5 @@
 <link name="ball_pusher">
   <visual>
-    <origin xyz="0 -0.025 0" rpy="0 0 0"/>
+    <origin xyz="0 -0.02 0" rpy="0 0 0"/>
     <geometry>
       <box size="0.025 0.01 0.025"/>

Commit message: Post Launch Update

File: arm2d2/arm2d2_description/urdf/base.urdf.xacro (robot description, xacro)
@@ -53,5 +53,4 @@
   <child link="base_link"/>
 </joint>
-<!--
 <link name="gripper_mount_l">
   <inertial>
@@ -67,10 +66,12 @@
     <material name="silver"/>
   </visual>
-  <collision>
-    <origin xyz="-0.0 3e-06 0.011329" rpy="0 0 0"/>
-    <geometry>
-      <mesh filename="package://arm2d2_description/meshes/gripper_mount.stl" scale="0.001 0.001 0.001"/>
-    </geometry>
-  </collision>
+  <!--
+  <collision>
+    <origin xyz="-0.0 3e-06 0.011329" rpy="0 0 0"/>
+    <geometry>
+      <mesh filename="package://arm2d2_description/meshes/gripper_mount.stl" scale="0.001 0.001 0.001"/>
+    </geometry>
+  </collision>
+  -->
 </link>
 <joint name="gripper_mount_l_joint" type="fixed">
@@ -92,10 +93,12 @@
     <material name="silver"/>
   </visual>
-  <collision>
-    <origin xyz="-0.0 3e-06 0.011329" rpy="0 0 0"/>
-    <geometry>
-      <mesh filename="package://arm2d2_description/meshes/gripper_mount.stl" scale="0.001 0.001 0.001"/>
-    </geometry>
-  </collision>
+  <!--
+  <collision>
+    <origin xyz="-0.0 3e-06 0.011329" rpy="0 0 0"/>
+    <geometry>
+      <mesh filename="package://arm2d2_description/meshes/gripper_mount.stl" scale="0.001 0.001 0.001"/>
+    </geometry>
+  </collision>
+  -->
 </link>
 <joint name="gripper_mount_r_joint" type="fixed">
@@ -104,5 +107,4 @@
   <child link="gripper_mount_r"/>
 </joint>
--->
 <!--
 <link name="soft_robotics">
@@ -119,6 +121,4 @@
   <child link="soft_robotics"/>
 </joint>
--->
-<!--
 <link name="camera_mount">
   <visual>

File: tundra_gripper/urdf/gripper.urdf.xacro (robot description, xacro)
@@ -29,4 +29,5 @@
     <child link="palm"/>
   </joint>
+<!-- Removed for catch training
 <link name="ball_pusher">
   <visual>
@@ -48,4 +49,5 @@
   <child link="ball_pusher"/>
 </joint>
+-->
   <link name="actuator_1">
     <inertial>
